File: 原理图+PCB/tuya_arduino/tuya_arduino.kicad_pcb (KiCad board)
At the start: 2 copper layers, 50 x 55 mm, 47 parts, among them J1 Conn_01x15_Male, J2 USB_A, J3 Conn_01x15_Male, J4 arduino_nano_base, J5 Conn_01x03_Female, J6 Conn_01x11_Male, J7 Conn_01x11_Male, J8 Conn_02x02_Top_Bottom_Mountin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, Q1 S8050, SW1 SW_Push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

Commit message: seconed commit
Parts:
- removed G***: LOGO, tuya_arduino:tuya-logo
- removed Q1: S8050, Package_TO_SOT_SMD:SOT-23
- removed R3, R6, R7: 2k, Resistor_SMD:R_0603_1608Metric_Pad0.98x0.95mm_HandSolder
- removed R5: NC/0R, Resistor_SMD:R_0603_1608Metric_Pad0.98x0.95mm_HandSolder
- removed REF**: HOLE_2MM, 0WJQ:HOLE_2MM
- removed REF**: KiCad-Logo_6mm_Copper, Symbol:KiCad-Logo_6mm_Copper
- removed REF**: MP_HOLE_L4_M3, 0WJQ:MP_HOLE_L4_M3
- added SW6: SW_DPST_x2, Button_Switch_SMD:SW_SPST_B3U-1000P, F.Cu at (82.5, 56.1)
- U2: footprint tuya_arduino:tuya_cbu -> 自用工程封装库:tuya_cbu
- moved J6 22.2 mm to (118.6, 96.5)
- moved J7 21.8 mm to (117.7, 74.3)
- moved U2 0.50 mm to (125.4, 77.7)
Connections:
- C1 pad 2: Net-(C1-Pad2) -> GND
- J2 pad 4: Net-(J2-Pad4) -> GND
- J3 pad 1: +5V -> /VIN
- J4 pad 30: +5V -> /VIN
- J7 pad 2: /OUT_RGB_TU_3V3 -> /OUT_RGB_TU
- R4 pad 1: /OUT_RGB_TU_5V -> /OUT_RGB_TU
- U2 pad 2: /OUT_RGB_TU_3V3 -> /OUT_RGB_TU
Routing:
- net +3V3: track 129.1 -> 52.6 mm, vias 2 -> 1
- net /OUT_RGB_TU_3V3: track 72.6 -> 0.00 mm
- net GND: track 78.4 -> 42.9 mm, vias 23 -> 21
- net /OUT_RGB_TU: track 0.00 -> 19.8 mm
- net +5V: track 125.1 -> 108.7 mm
- net /OUT_RGB_TU_5V: track 14.8 -> 0.00 mm
- net /TX_C: track 21.7 -> 35.8 mm
- net /RX_C: track 22.8 -> 36.7 mm
- net /P22: track 27.4 -> 37.4 mm, vias 0 -> 1
- net /VIN: track 0.00 -> 6.57 mm
- net /KEY_TU: track 41.2 -> 45.7 mm
- net /P24: track 18.0 -> 15.3 mm
- net /P26: track 21.0 -> 23.4 mm
- net (no net): track 0.00 -> 2.24 mm
- net Net-(Q1-Pad2): track 2.04 -> 0.00 mm
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