File: 原理图+PCB/tuya_arduino/tuya_arduino.sch (KiCad schematic (older format))
At the start: 43 parts, among them J1 Conn_01x15_Male, J2 USB_A, J3 Conn_01x15_Male, J4 arduino_nano_base, J5 Conn_01x03_Female, J6 Conn_01x11_Male, J7 Conn_01x11_Male, J8 Conn_02x02_Top_Bottom_Mountin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, Q1 S8050, SW1 SW_Push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

Commit message: seconed commit
Parts:
- removed Q1: S8050, Package_TO_SOT_SMD:SOT-23, symbol Transistor_BJT:S8050
- removed R3, R6, R7: 2k, Resistor_SMD:R_0603_1608Metric_Pad0.98x0.95mm_HandSolder, symbol Device:R
- removed R5: NC/0R, Resistor_SMD:R_0603_1608Metric_Pad0.98x0.95mm_HandSolder, symbol Device:R
- removed U2: mcu_tuya_cbu, tuya_arduino:tuya_cbu, symbol tuya_arduino_Library:mcu_tuya_cbu
- added SW6: SW_DPST_x2, Button_Switch_SMD:SW_SPST_B3U-1000P, symbol Switch:SW_DPST_x2
- added U2: mcu_tuya_cbu, 自用工程封装库:tuya_cbu, symbol 自用工程原理图库:mcu_tuya_cbu
Connections:
- net labels added: OUT_RGB_TU
- net labels removed: OUT_RGB_TU_3V3, OUT_RGB_TU_5V
- wire segments 219 -> 205
- no-connect marks 2 -> 5
Other:
- note removed: "level switching circuit"
- moved on the sheet: C10, C8, C9, D4, R2, SW4, SW5
